File: projects/microsd/microsd.kicad_pcb (KiCad board)
At the start: 2 copper layers, 20.3 x 12.7 mm, 7 parts, among them P1 CONN_8, P2 CONN_13, U1 74LS125

Commit message: minor changes
Parts:
- added VAL: REF, DIGITALCAVE_LOGO, B.Cu at (67.9, 36.8)
- added WJ10: VAL**, WJ10, B.Cu at (74.9, 36.8)
