File: projects/stubby/kicad/rev2.1/stubby.kicad_pcb (KiCad board)
At the start: 2 copper layers, 49.5 x 49.5 mm, 71 parts, among them IC1 ATMEGA1284-A, P1 CONN_6, P10 CONN_4, P11 CONN_6, P2 CONN_6, P3 CONN_10, P4 CONN_13, P5 CONN_4, P6 CONN_2, P7 CONN_1, P8 BATT (4.8V-6V), P9 PROG, SW1 SW_PUSH, SW2 DPDT, U1 HMC5883L, X1 CRYSTAL

Commit message: Re-annotated board
Parts:
- renumbered C7 to C10, C8 to C11, C9 to C12, C12 to C13, C19 to C14, C2 to C18, C3 to C2, C13 to C3, C14 to C5, C10 to C6, C11 to C7, C5 to C8, C6 to C9, P2 to P1, P5 to P2, P4 to P3, P6 to P4, P7 to P5, P1 to P6, P3 to P7, R9 to R10, R10 to R11, R11 to R8, R8 to R9, S2 to S1, S3 to S2, S4 to S3, S5 to S4, S6 to S5, S7 to S6, VR3 to VR2, VR2 to VR3
Changed lines of the file:
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@@
     (links 183)
     (no_connects 0)
-    (area 35.509999 14.554999 85.140001 64.185001)
+    (area 23.115001 13.74 86.865177 70.645)
     (thickness 1.6)
     (drawings 79)
@@
     (descr "Connecteur 10 pins")
     (tags "CONN DEV")
-    (fp_text reference P3 (at -6.35 -2.54) (layer F.SilkS) hide
+    (fp_text reference P7 (at -6.35 -2.54) (layer F.SilkS) hide
       (effects (font (size 1.72974 1.08712) (thickness 0.27178)))
     )
@@
     (at 58.42 29.21 180)
     (tags SOT23)
-    (fp_text reference VR3 (at 1.99898 -0.09906 270) (layer F.SilkS) hide
+    (fp_text reference VR2 (at 1.99898 -0.09906 270) (layer F.SilkS) hide
       (effects (font (size 0.762 0.762) (thickness 0.11938)))
     )
@@
     (descr "Connecteur 4 pibs")
     (tags "CONN DEV")
-    (fp_text reference P5 (at 0 -2.54) (layer F.SilkS) hide
+    (fp_text reference P2 (at 0 -2.54) (layer F.SilkS) hide
       (effects (font (size 1.73482 1.08712) (thickness 0.27178)))
     )
@@
     (descr "Connecteurs 2 pins")
     (tags "CONN DEV")
-    (fp_text reference P6 (at 0 -2.54) (layer F.SilkS) hide
+    (fp_text reference P4 (at 0 -2.54) (layer F.SilkS) hide
       (effects (font (size 1.72974 1.08712) (thickness 0.27178)))
     )
@@
     (descr "Connecteur 6 pins")
     (tags "CONN DEV")
-    (fp_text reference P2 (at 0 -2.54) (layer F.SilkS) hide
+    (fp_text reference P1 (at 0 -2.54) (layer F.SilkS) hide
       (effects (font (size 1.72974 1.08712) (thickness 0.27178)))
     )
@@
     (descr "Connecteurs 1 pin")
     (tags "CONN DEV")
-    (fp_text reference P7 (at 0 1.7) (layer B.SilkS) hide
+    (fp_text reference P5 (at 0 1.7) (layer B.SilkS) hide
       (effects (font (size 0.8 0.8) (thickness 0.15)) (justify mirror))
     )
@@
   (module HEX_LEG (layer F.Cu)
     (at 41.91 30.48 180)
-    (fp_text reference S4 (at -7.112 -1.524 270) (layer F.SilkS) hide
+    (fp_text reference S3 (at -7.112 -1.524 270) (layer F.SilkS) hide
       (effects (font (size 1 1) (thickness 0.15)))
     )
@@
   (module HEX_LEG (layer F.Cu)
     (at 41.91 21.59 180)
-    (fp_text reference S2 (at -7.112 -1.524 270) (layer F.SilkS) hide
+    (fp_text reference S1 (at -7.112 -1.524 270) (layer F.SilkS) hide
       (effects (font (size 1 1) (thickness 0.15)))
     )
@@
   (module HEX_LEG (layer F.Cu)
     (at 41.91 39.37 180)
-    (fp_text reference S6 (at -7.112 -1.524 270) (layer F.SilkS) hide
+    (fp_text reference S5 (at -7.112 -1.524 270) (layer F.SilkS) hide
       (effects (font (size 1 1) (thickness 0.15)))
     )
@@
   (module HEX_LEG_REVERSE (layer F.Cu)
     (at 78.74 25.4)
-    (fp_text reference S3 (at -8 -3 90) (layer F.SilkS) hide
+    (fp_text reference S2 (at -8 -3 90) (layer F.SilkS) hide
       (effects (font (size 1 1) (thickness 0.15)))
     )
@@
   (module HEX_LEG_REVERSE (layer F.Cu)
     (at 78.74 34.29)
-    (fp_text reference S5 (at -8 -3 90) (layer F.SilkS) hide
+    (fp_text reference S4 (at -8 -3 90) (layer F.SilkS) hide
       (effects (font (size 1 1) (thickness 0.15)))
     )
@@
   (module HEX_LEG_REVERSE (layer F.Cu)
     (at 78.74 43.18)
-    (fp_text reference S7 (at -8 -3 90) (layer F.SilkS) hide
+    (fp_text reference S6 (at -8 -3 90) (layer F.SilkS) hide
       (effects (font (size 1 1) (thickness 0.15)))
     )
@@
     (at 54.61 59.055)
     (tags "Bluetooth HC05 HC06")
-    (fp_text reference P4 (at -10.16 -2.54) (layer F.SilkS) hide
+    (fp_text reference P3 (at -10.16 -2.54) (layer F.SilkS) hide
       (effects (font (size 1.72974 1.08712) (thickness 0.27178)))
     )
@@
     (at 74.295 46.355 270)
     (attr smd)
-    (fp_text reference C7 (at 0 0 270) (layer F.SilkS) hide
+    (fp_text reference C10 (at 0 0 270) (layer F.SilkS) hide
       (effects (font (size 0.508 0.508) (thickness 0.1143)))
     )
@@
     (at 74.295 43.815 90)
     (attr smd)
-    (fp_text reference C8 (at 0 0 90) (layer F.SilkS) hide
+    (fp_text reference C11 (at 0 0 90) (layer F.SilkS) hide
       (effects (font (size 0.508 0.508) (thickness 0.1143)))
     )
@@
     (at 53.34 38.735)
     (attr smd)
-    (fp_text reference C5 (at 0 0) (layer F.SilkS) hide
+    (fp_text reference C8 (at 0 0) (layer F.SilkS) hide
       (effects (font (size 0.508 0.508) (thickness 0.1143)))
     )
@@
     (at 47.625 21.59)
     (attr smd)
-    (fp_text reference C3 (at 0 0) (layer F.SilkS) hide
+    (fp_text reference C2 (at 0 0) (layer F.SilkS) hide
       (effects (font (size 0.508 0.508) (thickness 0.1143)))
     )
@@
     (at 66.04 31.75 90)
     (attr smd)
-    (fp_text reference R8 (at 0 0 90) (layer F.SilkS) hide
+    (fp_text reference R9 (at 0 0 90) (layer F.SilkS) hide
       (effects (font (size 0.508 0.508) (thickness 0.1143)))
     )
@@
     (at 67.945 31.75 90)
     (attr smd)
-    (fp_text reference R10 (at 0 0 90) (layer F.SilkS) hide
+    (fp_text reference R11 (at 0 0 90) (layer F.SilkS) hide
       (effects (font (size 0.508 0.508) (thickness 0.1143)))
     )
@@
     (at 64.135 31.75 90)
     (attr smd)
-    (fp_text reference R9 (at 0 0 90) (layer F.SilkS) hide
+    (fp_text reference R10 (at 0 0 90) (layer F.SilkS) hide
       (effects (font (size 0.508 0.508) (thickness 0.1143)))
     )
@@
     (at 58.42 23.495)
     (attr smd)
-    (fp_text reference VR2 (at 2.19964 -0.29972 270) (layer F.SilkS) hide
+    (fp_text reference VR3 (at 2.19964 -0.29972 270) (layer F.SilkS) hide
       (effects (font (size 0.635 0.635) (thickness 0.127)))
     )
@@
     (at 53.34 29.845 180)
     (attr smd)
-    (fp_text reference C10 (at 0 0 180) (layer F.SilkS) hide
+    (fp_text reference C6 (at 0 0 180) (layer F.SilkS) hide
       (effects (font (size 0.762 0.762) (thickness 0.127)))
     )
@@
     (at 53.34 36.83)
     (attr smd)
-    (fp_text reference C12 (at 0 0) (layer F.SilkS) hide
+    (fp_text reference C13 (at 0 0) (layer F.SilkS) hide
       (effects (font (size 0.508 0.508) (thickness 0.1143)))
     )
@@
     (at 74.93 49.53 90)
     (attr smd)
-    (fp_text reference C6 (at 0 0 90) (layer F.SilkS) hide
+    (fp_text reference C9 (at 0 0 90) (layer F.SilkS) hide
       (effects (font (size 0.508 0.508) (thickness 0.1143)))
     )
@@
     (at 74.93 52.07)
     (attr smd)
-    (fp_text reference C9 (at 0 0) (layer F.SilkS) hide
+    (fp_text reference C12 (at 0 0) (layer F.SilkS) hide
       (effects (font (size 0.508 0.508) (thickness 0.1143)))
     )
@@
     (at 61.595 26.67)
     (attr smd)
-    (fp_text reference C13 (at 0 0) (layer F.SilkS) hide
+    (fp_text reference C3 (at 0 0) (layer F.SilkS) hide
       (effects (font (size 0.508 0.508) (thickness 0.1143)))
     )
@@
     (at 61.595 28.575)
     (attr smd)
-    (fp_text reference C14 (at 0 0) (layer F.SilkS) hide
+    (fp_text reference C5 (at 0 0) (layer F.SilkS) hide
       (effects (font (size 0.508 0.508) (thickness 0.1143)))
     )
@@
     (at 67.31 53.34)
     (attr smd)
-    (fp_text reference C19 (at 0 0) (layer F.SilkS) hide
+    (fp_text reference C14 (at 0 0) (layer F.SilkS) hide
       (effects (font (size 0.508 0.508) (thickness 0.1143)))
     )
@@
     (at 67.945 34.925 90)
     (attr smd)
-    (fp_text reference R11 (at 0 0 90) (layer F.SilkS) hide
+    (fp_text reference R8 (at 0 0 90) (layer F.SilkS) hide
       (effects (font (size 0.508 0.508) (thickness 0.1143)))
     )
@@
     (at 65.405 18.415 270)
     (descr "SMT capacitor, aluminium electrolytic, 5x5.3")
-    (fp_text reference C11 (at 0 -3.175 270) (layer F.SilkS) hide
+    (fp_text reference C7 (at 0 -3.175 270) (layer F.SilkS) hide
       (effects (font (size 0.50038 0.50038) (thickness 0.11938)))
     )
@@
     (descr "Connecteur 6 pins")
     (tags "CONN DEV")
-    (fp_text reference P1 (at 0 -2.54) (layer F.SilkS)
+    (fp_text reference P6 (at 0 -2.54) (layer F.SilkS)
       (effects (font (size 1.72974 1.08712) (thickness 0.3048)))
     )
@@
     (at 71.12 18.415 270)
     (descr "SMT capacitor, aluminium electrolytic, 5x5.3")
-    (fp_text reference C2 (at 0 -3.175 270) (layer F.SilkS) hide
+    (fp_text reference C18 (at 0 -3.175 270) (layer F.SilkS) hide
       (effects (font (size 0.50038 0.50038) (thickness 0.11938)))
     )
