File: projects/esc/esc.kicad_pcb (KiCad board)
At the start: 2 copper layers, 41 parts, among them IC1 ATMEGA48-A, P1 INPUT, P2 OUTPUT, Q1 Q_NMOS_GSD, Q2 Q_NMOS_GSD, Q3 Q_NMOS_GSD, Q4 Q_NMOS_GSD, Q5 Q_NMOS_GSD, Q6 Q_NMOS_GSD, U1 74LS08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

Commit message: fits into .5 x 3.9
Parts:
- added REF**: 1pin, Connect:1pin, F.Cu at (267.2, 97.2)
- added REF**: 1pin, Connect:1pin, F.Cu at (267.2, 106.2)
- added REF**: 1pin, Connect:1pin, F.Cu at (256.2, 101.6)
- added REF**: 1pin, Connect:1pin, F.Cu at (269.1, 101.6)
- moved R12 46.2 mm to (208.3, 101.6), turned to 270 degrees
- moved P1 17.1 mm to (178.4, 97.8)
- moved C3 16.5 mm to (204.5, 101.6), turned to 90 degrees
- moved MP2 15.9 mm to (186.1, 101.6)
- moved C2 11.9 mm to (189.2, 106.7), turned to 180 degrees
- moved C1 11.9 mm to (189.2, 96.5), turned to 180 degrees
- moved C4 8.35 mm to (191.1, 99.1)
- moved IC1 8.26 mm to (197.5, 101.6)
- moved C6 8.25 mm to (191.1, 104.1)
- moved C5 7.62 mm to (204.5, 104.8)
- moved C7 7.62 mm to (204.5, 98.4)
- moved R1 7.62 mm to (208.3, 104.8)
- moved R2 7.62 mm to (206.4, 104.8)
- moved R3 7.62 mm to (208.3, 98.4)
- moved R4 7.62 mm to (206.4, 98.4)
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Other:
- board outline added: 99.1 x 12.7 mm

Commit message: done routing for the night
Parts:
- moved C10 22.2 mm to (238.8, 96.5)
- moved R11 20.3 mm to (238.8, 98.4)
- moved Q4 8.52 mm to (251.5, 101.6)
- moved Q6 7.62 mm to (251.5, 105.4)
- moved Q3 5.85 mm to (243.8, 101.6)
- moved Q2 4.96 mm to (251.5, 97.8)
- moved P2 4.44 mm to (247.7, 99.1)
- moved Q1 4.44 mm to (243.8, 97.8)
- moved Q5 3.81 mm to (243.8, 105.4)
- moved REF** 1.17 mm to (266.4, 96.3)
- moved REF** 1.08 mm to (266.4, 106.9)
- moved IC1 0.63 mm to (197.5, 101.0)
- turned R18 to 0 degrees
Routing:
- net +BATT: track 0.00 -> 63.2 mm
- net Net-(Q2-Pad2): track 0.00 -> 28.2 mm
- net /U: track 0.00 -> 7.07 mm
- net /W: track 0.00 -> 6.28 mm
- net /V: track 0.00 -> 6.01 mm
Changed lines of the file:
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@@
   (general
     (links 100)
-    (no_connects 91)
+    (no_connects 79)
     (area 0 0 0 0)
     (thickness 1.6)
-    (drawings 16)
-    (tracks 18)
+    (drawings 12)
+    (tracks 49)
     (zones 0)
     (modules 45)
@@
   )
   (setup
-    (last_trace_width 0.25)
+    (last_trace_width 0.508)
+    (user_trace_width 0.254)
+    (user_trace_width 0.508)
     (trace_clearance 0.2)
     (zone_clearance 0.508)
@@
   )
   (module Connect:1pin (layer F.Cu)
-    (at 267.208 97.155)
+    (at 266.446 96.266)
     (descr "module 1 pin (ou trou mecanique de percage)")
     (tags DEV)
@@
   )
   (module Connect:1pin (layer F.Cu)
-    (at 267.208 106.172)
+    (at 266.446 106.934)
     (descr "module 1 pin (ou trou mecanique de percage)")
     (tags DEV)
@@
   )
   (module custom:SM0603_VALUE (layer F.Cu)
-    (at 218.44 105.41)
+    (at 238.76 96.52)
     (attr smd)
     (fp_text reference C10 (at 0 0) (layer F.SilkS) hide
@@
   )
   (module Housings_QFP:TQFP-32_7x7mm_Pitch0.8mm (layer F.Cu)
-    (at 197.485 101.6)
+    (at 197.485 100.965)
     (descr "32-Lead Plastic Thin Quad Flatpack (PT) - 7x7x1.0 mm Body, 2.00 mm [TQFP] (see Microchip Packaging Specification 00000049BS.pdf)")
     (tags "QFP 0.8")
@@
   )
   (module Pin_Headers:Pin_Header_Straight_1x03 (layer F.Cu)
-    (at 252.095 99.06)
+    (at 247.65 99.06)
     (descr "Through hole pin header")
     (tags "pin header")
@@
   )
   (module Housings_SOT-23_SOT-143_TSOT-6:SOT-23 (layer F.Cu)
-    (at 248.285 97.79 90)
+    (at 243.84 97.79 90)
     (descr "SOT-23, Standard")
     (tags SOT-23)
@@
   )
   (module Housings_SOT-23_SOT-143_TSOT-6:SOT-23 (layer F.Cu)
-    (at 248.285 101.6 90)
+    (at 251.46 97.79 90)
     (descr "SOT-23, Standard")
     (tags SOT-23)
@@
   )
   (module Housings_SOT-23_SOT-143_TSOT-6:SOT-23 (layer F.Cu)
-    (at 248.285 105.41 90)
+    (at 243.84 101.6 90)
     (descr "SOT-23, Standard")
     (tags SOT-23)
@@
   )
   (module Housings_SOT-23_SOT-143_TSOT-6:SOT-23 (layer F.Cu)
-    (at 243.84 97.79 90)
+    (at 251.46 101.6 90)
     (descr "SOT-23, Standard")
     (tags SOT-23)
@@
   )
   (module Housings_SOT-23_SOT-143_TSOT-6:SOT-23 (layer F.Cu)
-    (at 243.84 101.6 90)
+    (at 243.84 105.41 90)
     (descr "SOT-23, Standard")
     (tags SOT-23)
@@
   )
   (module Housings_SOT-23_SOT-143_TSOT-6:SOT-23 (layer F.Cu)
-    (at 243.84 105.41 90)
+    (at 251.46 105.41 90)
     (descr "SOT-23, Standard")
     (tags SOT-23)
@@
   )
   (module custom:SM0603_VALUE (layer F.Cu)
-    (at 218.44 97.79)
+    (at 238.76 98.425)
     (attr smd)
     (fp_text reference R11 (at 0 0) (layer F.SilkS) hide
@@
   )
   (module custom:RESISTOR_POWER (layer F.Cu)
-    (at 228.6 101.6 180)
-    (fp_text reference R18 (at 0 -3 180) (layer F.SilkS) hide
-      (effects (font (size 1 1) (thickness 0.15)))
-    )
-    (fp_text value 0.1 (at -5 2 180) (layer F.SilkS)
+    (at 228.6 101.6)
+    (fp_text reference R18 (at 0 -3) (layer F.SilkS) hide
+      (effects (font (size 1 1) (thickness 0.15)))
+    )
+    (fp_text value 0.1 (at -5 2) (layer F.SilkS)
       (effects (font (size 1 1) (thickness 0.15)))
     )
@@
     (fp_line (start 5 2) (end 6 0) (layer F.SilkS) (width 0.15))
     (fp_line (start 6 0) (end 8 0) (layer F.SilkS) (width 0.15))
-    (pad 1 thru_hole circle (at -10 0 180) (size 3.048 3.048) (drill 1.524) (layers *.Cu *.Mask F.SilkS)
-      (net 2 GND))
-    (pad 2 thru_hole circle (at 10 0 180) (size 3.048 3.048) (drill 1.524) (layers *.Cu *.Mask F.SilkS)
+    (pad 1 thru_hole circle (at -10 0) (size 3.048 3.048) (drill 1.524) (layers *.Cu *.Mask F.SilkS)
+      (net 2 GND))
+    (pad 2 thru_hole circle (at 10 0) (size 3.048 3.048) (drill 1.524) (layers *.Cu *.Mask F.SilkS)
       (net 38 "Net-(Q2-Pad2)"))
   )
@@
   )
   (gr_line (start 271.145 101.6) (end 147.32 101.6) (angle 90) (layer Cmts.User) (width 0.2))
-  (gr_circle (center 267.058349 97.14638) (end 267.058349 98.146378) (layer Cmts.User) (width 0.2))
-  (gr_circle (center 267.058349 106.14638) (end 267.05835 107.146378) (layer Cmts.User) (width 0.2))
-  (gr_circle (center 256.05835 101.646379) (end 256.058349 102.646378) (layer Cmts.User) (width 0.2))
-  (gr_circle (center 269.05835 101.646379) (end 269.05835 102.646378) (layer Cmts.User) (width 0.2))
   (gr_circle (center 262.558349 101.64638) (end 262.558349 109.646378) (layer Cmts.User) (width 0.2))
+  (segment (start 189.23 106.68) (end 189.865 107.315) (width 0.508) (layer F.Cu) (net 1))
+  (segment (start 189.865 107.315) (end 242.57 107.315) (width 0.508) (layer F.Cu) (net 1))
+  (segment (start 242.57 107.315) (end 242.84178 107.04322) (width 0.508) (layer F.Cu) (net 1))
+  (segment (start 242.84178 107.04322) (end 242.84178 105.41) (width 0.508) (layer F.Cu) (net 1))
+  (segment (start 242.84178 97.79) (end 242.84178 101.6) (width 0.508) (layer F.Cu) (net 1))
+  (segment (start 242.84178 105.41) (end 242.84178 101.6) (width 0.508) (layer F.Cu) (net 1))
   (segment (start 211.455 105.537) (end 213.36 105.537) (width 0.25) (layer F.Cu) (net 2))
   (segment (start 211.455 105.537) (end 210.312 105.537) (width 0.25) (layer F.Cu) (net 2))
@@
   (segment (start 213.36 104.013) (end 215.265 104.013) (width 0.25) (layer F.Cu) (net 10))
   (segment (start 211.455 104.013) (end 213.36 104.013) (width 0.25) (layer F.Cu) (net 10))
+  (segment (start 250.46178 97.79) (end 248.92 97.79) (width 0.508) (layer F.Cu) (net 33))
+  (segment (start 248.92 97.79) (end 247.65 99.06) (width 0.508) (layer F.Cu) (net 33))
+  (segment (start 244.84076 96.84) (end 245.43 96.84) (width 0.508) (layer F.Cu) (net 33))
+  (segment (start 245.43 96.84) (end 247.65 99.06) (width 0.508) (layer F.Cu) (net 33))
+  (segment (start 250.46178 101.6) (end 247.65 101.6) (width 0.508) (layer F.Cu) (net 34))
+  (segment (start 244.84076 100.65) (end 246.7 100.65) (width 0.508) (layer F.Cu) (net 34))
+  (segment (start 246.7 100.65) (end 247.65 101.6) (width 0.508) (layer F.Cu) (net 34))
+  (segment (start 247.65 104.14) (end 249.19178 104.14) (width 0.508) (layer F.Cu) (net 35))
+  (segment (start 249.19178 104.14) (end 250.46178 105.41) (width 0.508) (layer F.Cu) (net 35))
+  (segment (start 244.84076 104.46) (end 247.33 104.46) (width 0.508) (layer F.Cu) (net 35))
+  (segment (start 247.33 104.46) (end 247.65 104.14) (width 0.508) (layer F.Cu) (net 35))
+  (segment (start 252.46076 96.84) (end 252.415 96.84) (width 0.508) (layer F.Cu) (net 38))
+  (segment (start 252.415 96.84) (end 251.46 95.885) (width 0.508) (layer F.Cu) (net 38))
+  (segment (start 240.665 99.535) (end 238.6 101.6) (width 0.508) (layer F.Cu) (net 38))
+  (segment (start 240.665 97.155) (end 240.665 99.535) (width 0.508) (layer F.Cu) (net 38))
+  (segment (start 241.935 95.885) (end 240.665 97.155) (width 0.508) (layer F.Cu) (net 38))
+  (segment (start 251.46 95.885) (end 241.935 95.885) (width 0.508) (layer F.Cu) (net 38))
+  (segment (start 252.46076 100.65) (end 254 99.11076) (width 0.508) (layer F.Cu) (net 38))
+  (segment (start 254 99.11076) (end 254 98.425) (width 0.508) (layer F.Cu) (net 38))
+  (segment (start 254 98.425) (end 252.46076 96.88576) (width 0.508) (layer F.Cu) (net 38))
+  (segment (start 252.46076 96.88576) (end 252.46076 96.84) (width 0.508) (layer F.Cu) (net 38))
+  (segment (start 252.46076 100.65) (end 252.46076 100.69576) (width 0.508) (layer F.Cu) (net 38))
+  (segment (start 252.46076 100.69576) (end 254 102.235) (width 0.508) (layer F.Cu) (net 38))
+  (segment (start 254 102.92076) (end 252.46076 104.46) (width 0.508) (layer F.Cu) (net 38))
+  (segment (start 254 102.235) (end 254 102.92076) (width 0.508) (layer F.Cu) (net 38))
 )

Commit message: wip
Parts:
- removed C10: 2.2n, custom:SM0603_VALUE
- removed C11, C7, C8, C9: C_Small, custom:SM0603_VALUE
- removed C3: 4.7n, custom:SM0603_VALUE
- removed C4, C5, C6: 0.1u, custom:SM0603_VALUE
- removed IC1: ATMEGA48-A, Housings_QFP:TQFP-32_7x7mm_Pitch0.8mm
- removed R10, R15, R4, R8: 5.1k, custom:SM0603_VALUE
- removed R11, R12, R14, R3, R7, R9: 10k, custom:SM0603_VALUE
- removed R13, R5, R6: 1k, custom:SM0603_VALUE
- removed R18: 0.1, custom:RESISTOR_POWER
- removed REF** (x4): 1pin, Connect:1pin
- removed U2: 74LS08, Housings_SSOP:SSOP-14_5.3x6.2mm_Pitch0.65mm
- C1: footprint Capacitors_ThroughHole:C_Radial_D5_L6_P2.5 -> Capacitors_SMD:C_0603
- C2: value 220u -> CP1
- D1: value RGB_LED_COMMON_ANODE_ALT1 -> LED; footprint custom:LED_RGB_4-PLCC_ALT1 -> LEDs:LED-0603
- Q1, Q3, Q5: value Q_NMOS_GSD -> Q_PMOS_GSD
- R1: value 10k -> R_Small
- R2: value 5.1k -> RESISTOR; footprint custom:SM0603_VALUE -> Resistors_SMD:R_2512
- U1: value 74LS08 -> CONN_01X20; footprint Housings_SSOP:SSOP-14_5.3x6.2mm_Pitch0.65mm -> Housings_SSOP:TSSOP-20_4.4x6.5mm_Pitch0.65mm
- moved C1 83.3 mm to (272.4, 101.7), turned to 270 degrees
- moved R2 45.2 mm to (251.5, 101.7)
- moved MP1 24.8 mm to (179.7, 101.6)
- moved C2 12.5 mm to (200.0, 100.3), turned to 270 degrees
- moved MP2 7.62 mm to (193.7, 101.6)
- moved P1 6.98 mm to (185.4, 97.8)
- moved U1 5.72 mm to (219.1, 101.6), turned to 0 degrees
- moved P2 5.10 mm to (242.5, 99.1)
- moved Q1 5.10 mm to (238.7, 97.8)
- moved Q2 5.10 mm to (246.4, 97.8)
- moved Q3 5.10 mm to (238.7, 101.6)
- moved Q4 5.10 mm to (246.4, 101.6)
- moved Q5 5.10 mm to (238.7, 105.4)
- moved Q6 5.10 mm to (246.4, 105.4)
- moved R1 1.28 mm to (209.6, 104.6)
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Connections:
- D1 pad 1: +3V3 -> Net-(D1-Pad1)
- D1 pad 2: Net-(D1-Pad2) -> +BATT
- P1 pad 1: /MISO -> /SDO
- P1 pad 2: +3V3 -> +BATT
- P1 pad 3: /SCLK -> /SCK
- P1 pad 4: /MOSI -> /FAULT
- P1 pad 5: /RESET -> /STR
- P1 pad 6: GND -> /SPD
- P1 pad 7: /SEL -> /SDI
- P1 pad 8: +BATT -> GND
- P2 pad 1: /U -> /SA
- P2 pad 2: /V -> /SB
- P2 pad 3: /W -> /SC
- Q1 pad 1: /UH_PWM -> /GHA
- Q1 pad 2: /U -> /SA
- Q2 pad 1: /UL_PWM -> /GLA
- Q2 pad 2: Net-(Q2-Pad2) -> /CSP
- Q2 pad 3: /U -> /SA
- Q3 pad 1: /VH_PWM -> /GHB
- Q3 pad 2: /V -> /SB
- Q4 pad 1: /VL_PWM -> /GLB
- Q4 pad 2: Net-(Q2-Pad2) -> /CSP
- Q4 pad 3: /V -> /SB
- Q5 pad 1: /WH_PWM -> /GHC
- Q5 pad 2: /W -> /SC
- Q6 pad 1: /WL_PWM -> /GLC
- Q6 pad 2: Net-(Q2-Pad2) -> /CSP
- Q6 pad 3: /W -> /SC
- R1 pad 1: +3V3 -> GND
- R1 pad 2: Net-(C3-Pad1) -> Net-(D1-Pad1)
- R2 pad 1: Net-(C3-Pad1) -> /CSP
- U1 pad 1: /PWM_OUT -> +BATT
- U1 pad 10: /UH_EN -> GND
- U1 pad 11: (no net) -> /CSP
- U1 pad 12: (no net) -> /GLC
- U1 pad 13: (no net) -> /GLB
- U1 pad 14: +3V3 -> /GLA
- U1 pad 2: /WH_EN -> /FAULT
- U1 pad 3: /WH_PWM -> /SPD
- U1 pad 4: /PWM_OUT -> /FAULT
- U1 pad 5: /VH_EN -> /SDO
- U1 pad 6: /VH_PWM -> /SCK
- U1 pad 7: GND -> /STR
- U1 pad 8: /UH_PWM -> /SDI
- U1 pad 9: /PWM_OUT -> GND
Routing:
- net +BATT: track 63.2 -> 7.62 mm
- net Net-(Q2-Pad2): track 28.2 -> 0.00 mm
- net /CSP: track 0.00 -> 17.9 mm
- net GND: track 9.68 -> 0.00 mm, vias 3 -> 0
- net /U: track 7.07 -> 0.00 mm
- net /SA: track 0.00 -> 7.07 mm
- net /W: track 6.28 -> 0.00 mm
- net /SC: track 0.00 -> 6.28 mm
- net /V: track 6.01 -> 0.00 mm
- net /SB: track 0.00 -> 6.01 mm
- net /W_REF: track 3.81 -> 0.00 mm
- net /V_REF: track 3.81 -> 0.00 mm
- net /U_REF: track 3.81 -> 0.00 mm
- added copper zone on B.Cu, net +BATT
- added copper zone on F.Cu, net +BATT
- added copper zone on B.Cu, net GND
