File: projects/m16/kicad/arm/m16.sch (KiCad schematic (older format))
At the start: 44 parts, among them J1 TST, J2 SWD, J3 Peripheral, J4 ESP8266, J5 Molex 475710001, J6 CONN_01X02, J7 HUB75, J8 Power, Q1 BSS138, U1 STM32F411RETx, U2 LM1117-3.3, U3 24LC16, Y1 ABS25-32.768-6

Commit message: wip
Parts:
- added C4: C, Capacitors_SMD:C_0603, symbol C
- BT1: value 3V -> 2032 3V
- J3: footprint (none) -> Pin_Headers:Pin_Header_Straight_2x06_Pitch2.54mm
- J4: footprint (none) -> Pin_Headers:Pin_Header_Straight_2x04_Pitch2.54mm
Connections:
- wire segments 120 -> 122

Commit message: got board layed out again
Parts:
- removed J1: TST, Pin_Headers:Pin_Header_Straight_1x01_Pitch1.27mm, symbol Conn_01x01
- removed J3: Peripheral, Pin_Headers:Pin_Header_Straight_2x06_Pitch2.54mm, symbol Conn_02x06_Odd_Even
- removed J6: CONN_01X02, Pin_Headers:Pin_Header_Straight_1x02_Pitch2.54mm, symbol Conn_01x02
- removed J8: Power, Connectors_Phoenix:PhoenixContact_MSTBVA-G_02x5.00mm_Vertical, symbol Conn_02x01
- added D2: D_TVS_x2_AAC, TO_SOT_Packages_SMD:SOT-23, symbol D_TVS_x2_AAC
- added J1: ENCODER, Pin_Headers:Pin_Header_Straight_1x02_Pitch2.54mm, symbol Conn_01x02
- added J10: IR, Pin_Headers:Pin_Header_Straight_1x03_Pitch2.54mm, symbol Conn_01x03
- added J11: WS2812, Pin_Headers:Pin_Header_Straight_1x03_Pitch2.54mm, symbol Conn_01x03
- added J3: BUTTONS, Pin_Headers:Pin_Header_Straight_2x02_Pitch2.54mm, symbol Conn_02x02_Counter_Clockwise
- added J6: FTDI, Pin_Headers:Pin_Header_Straight_1x06_Pitch2.54mm, symbol Conn_01x06
- added J8: POWER, Connectors:BARREL_JACK, symbol Barrel_Jack
- added J9: PIEZO, Pin_Headers:Pin_Header_Straight_1x02_Pitch2.54mm, symbol Conn_01x02
- added Q2: BSS138, TO_SOT_Packages_SMD:SOT-23, symbol BSS138
- added R15: 100, Resistors_SMD:R_0603, symbol R_Small
- added R16: 10k, Resistors_SMD:R_0603, symbol R_Small
- added R2, R4: 1k, Resistors_SMD:R_0603, symbol R_Small
Connections:
- net labels added: ESP_EN, ESP_RX, ESP_TX, FTDI_RX, FTDI_TX, IR_DO, WS_DI
- net labels removed: EN1A, EN1B, RX_TX, SD_DET, TST, TX_RX, WS_D33
- wire segments 122 -> 147
- no-connect marks 24 -> 30
Other:
- note removed: "EN"
- note removed: "ENCODER"
- note removed: "ENCODERS"
- note removed: "GND"
- note removed: "RST"
- note removed: "RX"
- note removed: "TX"
- note removed: "VCC"

Commit message: cleaning up and labeling board
Parts:
- C4: value C -> 100n
- J1: value ENCODER -> ENCR
- J3: value BUTTONS -> BTNS
Changed lines of the file:
@@
 P 4500 1200
 F 0 "C4" H 4525 1300 50  0000 L CNN
-F 1 "C" H 4525 1100 50  0000 L CNN
+F 1 "100n" H 4525 1100 50  0000 L CNN
 F 2 "Capacitors_SMD:C_0603" H 4538 1050 50  0001 C CNN
 F 3 "" H 4500 1200 50  0001 C CNN
@@
 P 700 6600
 F 0 "J1" H 700 6700 50  0000 C CNN
-F 1 "ENCODER" H 700 6400 50  0000 C CNN
+F 1 "ENCR" H 700 6400 50  0000 C CNN
 F 2 "Pin_Headers:Pin_Header_Straight_1x02_Pitch2.54mm" H 700 6600 50  0001 C CNN
 F 3 "" H 700 6600 50  0001 C CNN
@@
 P 1550 4800
 F 0 "J3" H 1600 4900 50  0000 C CNN
-F 1 "BUTTONS" H 1600 4600 50  0000 C CNN
+F 1 "BTNS" H 1600 4600 50  0000 C CNN
 F 2 "Pin_Headers:Pin_Header_Straight_2x02_Pitch2.54mm" H 1550 4800 50  0001 C CNN
 F 3 "" H 1550 4800 50  0001 C CNN

Commit message: wip level shifters
Parts:
- removed J2: SWD, Pin_Headers:Pin_Header_Straight_1x06_Pitch2.54mm, symbol Conn_01x06
- removed J6: FTDI, Pin_Headers:Pin_Header_Straight_1x06_Pitch2.54mm, symbol Conn_01x06
- removed Q1: BSS138, TO_SOT_Packages_SMD:SOT-23, symbol BSS138
- removed R10, R12: 10K, Resistors_SMD:R_0603, symbol R_Small
- added C17, C2: 100n, Capacitors_SMD:C_0603, symbol C_Small
- added J2: SWD, Pin_Headers:Pin_Header_Straight_1x08_Pitch2.54mm, symbol Conn_01x08
- added U4, U5: 74HCT244, Housings_SSOP:TSSOP-20_4.4x6.5mm_Pitch0.65mm, symbol 74HCT244
Connections:
- net labels added: IDC_A, IDC_B, IDC_B0, IDC_B1, IDC_C, IDC_CLK, IDC_D, IDC_G0, IDC_G1, IDC_OE, IDC_R0, IDC_R1, IDC_STB, RGB_A, RGB_B, RGB_B0, RGB_B1, RGB_C, RGB_D, RGB_G0, RGB_G1, RGB_R0, RGB_R1, RX, TX
- net labels removed: A, B, B0, B1, C, D, FTDI_RX, FTDI_TX, G0, G1, R0, R1
- wire segments 147 -> 151
- no-connect marks 30 -> 32
Other:
- note added: "ENCODER"
- note added: "IR"
- note added: "LEVEL SHIFT"
- note added: "RTC CRYSTAL"
- note added: "SD CARD"
- note added: "SWITCHES"
- note added: "WIFI"
- note added: "WS2812"

Commit message: finished rerouting pcb
Parts:
- added J6: Conn_01x02, DigitalCave:SCREW_TERMINAL_2, symbol Conn_01x02
Connections:
- wire segments 151 -> 153
Changed lines of the file:
@@
 NoConn ~ 10700 5250
 NoConn ~ 9700 5250
+$Comp
+L Conn_01x02 J6
+U 1 1 5BF167B3
+P 8750 1450
+F 0 "J6" H 8750 1550 50  0000 C CNN
+F 1 "Conn_01x02" H 8750 1250 50  0000 C CNN
+F 2 "DigitalCave:SCREW_TERMINAL_2" H 8750 1450 50  0001 C CNN
+F 3 "" H 8750 1450 50  0001 C CNN
+	1    8750 1450
+	1    0    0    -1
+$EndComp
+$Comp
+L +5V #PWR049
+U 1 1 5BF16C9E
+P 8450 1450
+F 0 "#PWR049" H 8450 1300 50  0001 C CNN
+F 1 "+5V" H 8450 1590 50  0000 C CNN
+F 2 "" H 8450 1450 50  0001 C CNN
+F 3 "" H 8450 1450 50  0001 C CNN
+	1    8450 1450
+	1    0    0    -1
+$EndComp
+$Comp
+L GND #PWR050
+U 1 1 5BF16D4E
+P 8450 1550
+F 0 "#PWR050" H 8450 1300 50  0001 C CNN
+F 1 "GND" H 8450 1400 50  0000 C CNN
+F 2 "" H 8450 1550 50  0001 C CNN
+F 3 "" H 8450 1550 50  0001 C CNN
+	1    8450 1550
+	1    0    0    -1
+$EndComp
+Wire Wire Line
+	8550 1450 8450 1450
+Wire Wire Line
+	8550 1550 8450 1550
 $EndSCHEMATC

Commit message: adding led, fixing sdio_cmd
Parts:
- added D3: LED, LEDs:LED_0603, symbol LED
- added R10: 68, Resistors_SMD:R_0603, symbol R_Small
Connections:
- net labels added: LED
- no-connect marks 32 -> 31
Changed lines of the file:
@@
 	0    -1   -1   0
 $EndComp
-Text Label 8600 3550 0    60   ~ 0
+Text Label 8650 2900 0    60   ~ 0
 SDIO_CMD
 $Comp
@@
 	-1   0    0    1
 $EndComp
-Text Label 8750 4600 0    60   ~ 0
+Text Label 8650 4600 0    60   ~ 0
 SCL
-Text Label 8750 4700 0    60   ~ 0
+Text Label 8650 4700 0    60   ~ 0
 SDA
 Text Label 1150 3400 2    60   ~ 0
@@
 	5500 800  5500 700
 Wire Wire Line
-	8650 4600 8750 4600
-Wire Wire Line
-	8650 4700 8750 4700
-Wire Wire Line
 	1150 5100 1700 5100
 Wire Wire Line
@@
 NoConn ~ 8650 4100
 NoConn ~ 2850 5200
-NoConn ~ 2850 3700
 NoConn ~ 8650 3100
 NoConn ~ 1300 2050
@@
 Wire Wire Line
 	8550 1550 8450 1550
+$Comp
+L LED D3
+U 1 1 5BF1CBE9
+P 7750 6100
+F 0 "D3" H 7750 6200 50  0000 C CNN
+F 1 "LED" H 7750 6000 50  0000 C CNN
+F 2 "LEDs:LED_0603" H 7750 6100 50  0001 C CNN
+F 3 "" H 7750 6100 50  0001 C CNN
+	1    7750 6100
+	1    0    0    -1
+$EndComp
+Text Label 7900 6100 0    60   ~ 0
+LED
+$Comp
+L R_Small R10
+U 1 1 5BF1CF60
+P 7400 6100
+F 0 "R10" H 7430 6120 50  0000 L CNN
+F 1 "68" H 7430 6060 50  0000 L CNN
+F 2 "Resistors_SMD:R_0603" H 7400 6100 50  0001 C CNN
+F 3 "" H 7400 6100 50  0001 C CNN
+	1    7400 6100
+	0    1    1    0
+$EndComp
+$Comp
+L GND #PWR051
+U 1 1 5BF1D0D7
+P 7200 6100
+F 0 "#PWR051" H 7200 5850 50  0001 C CNN
+F 1 "GND" H 7200 5950 50  0000 C CNN
+F 2 "" H 7200 6100 50  0001 C CNN
+F 3 "" H 7200 6100 50  0001 C CNN
+	1    7200 6100
+	0    1    1    0
+$EndComp
+Wire Wire Line
+	7200 6100 7300 6100
+Wire Wire Line
+	7500 6100 7600 6100
+Text Label 2850 3700 2    60   ~ 0
+LED
 $EndSCHEMATC

Commit message: complete overhaul of PCB
Parts:
- removed J2: SWD, Pin_Headers:Pin_Header_Straight_1x08_Pitch2.54mm, symbol Conn_01x08
- removed MP1, MP2: MOUNTING_HOLE, DigitalCave:MOUNTING_HOLE_#4, symbol MOUNTING_HOLE
- removed Q2: BSS138, TO_SOT_Packages_SMD:SOT-23, symbol BSS138
- added C19, C20: 8p, Capacitors_SMD:C_0603, symbol C_Small
- added J12: USB_OTG, Connectors_USB:USB_Micro-B_Molex_47346-0001, symbol USB_OTG
- added J13: SERIAL, Pin_Headers:Pin_Header_Straight_1x02_Pitch2.54mm, symbol Conn_01x02
- added J2: SWD, Pin_Headers:Pin_Header_Straight_1x06_Pitch2.54mm, symbol Conn_01x06
- added Q1: MMBT3904, TO_SOT_Packages_SMD:SOT-23, symbol MMBT3904
- added R12, R17: 22, Resistors_SMD:R_0603, symbol R_Small
- added Y2: 16MHz, Crystals:Crystal_SMD_0603-2pin_6.0x3.5mm, symbol Crystal
Connections:
- net labels added: HSE_N, HSE_P, LSE_N, LSE_P, USB_DM, USB_DP
- net labels removed: IR_DI, OSC32_N, OSC32_P
- wire segments 153 -> 158
- no-connect marks 31 -> 28

Commit message: adding solder bridge on vbus
Parts:
- added J14: GS2, Connectors:GS2, symbol GS2
Connections:
- wire segments 158 -> 159
